Commit message: added lidars and cleaned some files

File: kmr_iiwa_gazebo/urdf/kmr_iiwa.urdf.xacro (robot description, xacro)
@@ -18,5 +18,5 @@
       default="$(find lbr_ros2_control)/config/initial_joint_positions.yaml" />
   <!-- ROBOT -->
-  <xacro:kuka_kmp200 prefix="$(arg base_name)"/>
+  <xacro:kuka_kmp200 base_name="$(arg base_name)"/>
   <xacro:lbr_iiwa14_r820
     robot_name="$(arg robot_name)"/>
@@ -66,3 +66,71 @@
   <link name="world"/>
   <xacro:virtual_base_system world_link="world" base_link="$(arg base_name)_base_link" />
+  <!-- Sensors -->
+  <gazebo reference="$(arg base_name)_lidar_front_right_link">
+  <sensor name="lidar_front_right" type="gpu_lidar">
+      <pose relative_to='$(arg base_name)_lidar_front_right_link'>0 0 0 0 0 0</pose>
+      <topic>$(arg robot_name)/lidar_front_right</topic>
+      <gz_frame_id>$(arg base_name)_lidar_front_right_link</gz_frame_id>
+      <!-- Response time 80 ms -->
+      <update_rate>12.5</update_rate>
+      <always_on>1</always_on>
+      <visualize>true</visualize>
+      <ray>
+        <scan>
+          <horizontal>
+              <samples>540</samples>
+              <resolution>1</resolution>
+              <!-- avoid the base -->
+              <min_angle>-2</min_angle>
+              <max_angle>2</max_angle>
+          </horizontal>
+          <vertical>
+              <samples>1</samples>
+              <resolution>0.01</resolution>
+              <min_angle>0</min_angle>
+              <max_angle>0</max_angle>
+          </vertical>
+        </scan>
+        <range>
+            <min>0.05</min>
+            <max>30.0</max>
+            <!-- Resolution (can be configured) 30 mm, 40 mm, 50 mm, 70 mm, 150 mm -->
+            <resolution>0.05</resolution>
+        </range>
+    </ray>
+  </sensor>
+  </gazebo>
+  <gazebo reference="$(arg base_name)_lidar_back_left_link">
+  <sensor name="lidar_back_left" type="gpu_lidar">
+      <pose relative_to='$(arg base_name)_lidar_back_left_link'>0 0 0 0 0 0</pose>
+      <topic>$(arg robot_name)/lidar_back_left</topic>
+      <gz_frame_id>$(arg base_name)_lidar_back_left_link</gz_frame_id>
+      <!-- Response time 80 ms -->
+      <update_rate>12.5</update_rate>
+      <always_on>1</always_on>
+      <visualize>true</visualize>
+      <ray>
+        <scan>
+          <horizontal>
+              <samples>540</samples>
+              <resolution>1</resolution>
+              <min_angle>-2</min_angle>
+              <max_angle>2</max_angle>
+          </horizontal>
+          <vertical>
+              <samples>1</samples>
+              <resolution>0.01</resolution>
+              <min_angle>0</min_angle>
+              <max_angle>0</max_angle>
+          </vertical>
+        </scan>
+        <range>
+            <min>0.05</min>
+            <max>30.0</max>
+            <!-- Resolution (can be configured) 30 mm, 40 mm, 50 mm, 70 mm, 150 mm -->
+            <resolution>0.05</resolution>
+        </range>
+    </ray>
+  </sensor>
+  </gazebo>
 </robot>

File: kmr_iiwa_urdf/urdf/kmp200_macro.urdf.xacro (robot description, xacro)
@@ -3,6 +3,6 @@
   <!-- include helper xacros -->
   <xacro:include filename="$(find kmr_iiwa_urdf)/urdf/common_materials.xacro"/>
-  <xacro:macro name="kuka_kmp200" params="prefix">
-  <link name="${prefix}_base_link">
+  <xacro:macro name="kuka_kmp200" params="base_name">
+  <link name="${base_name}_base_link">
     <inertial>
     <origin xyz="0 0 0.35" rpy="0 0 0"/>
@@ -31,4 +31,17 @@
     </collision>
   </link>
+  <!-- laser Scanner laserscanner S300 optic-->
+  <joint name="${base_name}_lidar_front_right_joint" type="fixed">
+      <parent link="${base_name}_base_link" />
+      <child link="${base_name}_lidar_front_right_link" />
+      <origin xyz="0.464 -0.256 0.15" rpy="0 0 -0.7854"/>
+  </joint>
+  <link name="${base_name}_lidar_front_right_link"></link>
+  <joint name="${base_name}_lidar_back_left_joint" type="fixed">
+      <parent link="${base_name}_base_link" />
+      <child link="${base_name}_lidar_back_left_link" />
+      <origin xyz="-0.464 0.256 0.15" rpy="0 0 2.3562"/>
+  </joint>
+  <link name="${base_name}_lidar_back_left_link"></link>
   </xacro:macro>
 </robot>

Commit message: odom root frame better for nav2, but fake inertia necessary

File: kmr_iiwa_gazebo/urdf/kmr_iiwa.urdf.xacro (robot description, xacro)
@@ -64,6 +64,14 @@
   </ros2_control> -->
   <!-- OPTION 3. virtual joints, virtual base system -->
-  <link name="world"/>
-  <xacro:virtual_base_system world_link="world" base_link="$(arg base_name)_base_link" />
+  <link name="odom">
+    <inertial>
+      <mass value="0.001"/>
+      <inertia
+        ixx="1e-6" ixy="0" ixz="0"
+        iyy="1e-6" iyz="0"
+        izz="1e-6"/>
+    </inertial>
+  </link>
+  <xacro:virtual_base_system world_link="odom" base_link="$(arg base_name)_base_link" />
   <!-- Sensors -->
   <gazebo reference="$(arg base_name)_lidar_front_right_link">
